File: akiduki_headphone_amp.kicad_sch (KiCad schematic)
At the start: 22 parts, among them J1 IN, J2 OUT, U1 NJM4558

Commit message: パーツ間を詰めた
Parts:
- added H1, H2, H3, H4: MountingHole, MountingHole:MountingHole_3.2mm_M3, symbol Mechanical:MountingHole
